File: boards/se/pds.kicad_sch (KiCad schematic)
At the start: 1 part, among them J1 SE_PDS

Commit message: Schematic PDFs
Parts:
- J1: value SE_PDS -> Macintosh SE PDS Interface; footprint PDS_Connector:DIN41612_C_3x40_Male_Horizontal_THT -> Connector_DIN:DIN41612_C_3x32_Female_Vertical_THT
Changed lines of the file:
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@@
   (symbol (lib_id "PDS-Ethernet:SE_PDS") (at 68.58 27.94 0) (unit 1)
     (in_bom yes) (on_board yes) (dnp no) (fields_autoplaced)
-    (property "Reference" "J1" (at 90.8559 30.48 0)
+    (property "Reference" "J1" (at 87.0459 135.89 0)
       (effects (font (size 1.27 1.27)) (justify left))
     )
-    (property "Value" "SE_PDS" (at 90.8559 33.02 0)
+    (property "Value" "Macintosh SE PDS Interface" (at 87.0459 138.43 0)
       (effects (font (size 1.27 1.27)) (justify left))
     )
-    (property "Footprint" "PDS_Connector:DIN41612_C_3x40_Male_Horizontal_THT" (at 177.8 21.59 0)
+    (property "Footprint" "Connector_DIN:DIN41612_C_3x32_Female_Vertical_THT" (at 177.8 21.59 0)
       (effects (font (size 1.27 1.27)) hide)
     )

Commit message: Rev1 hardware
Parts:
- J1: footprint Connector_DIN:DIN41612_C_3x32_Female_Vertical_THT -> PDS-Ethernet:DIN41612_C_3x32_Female_Vertical_THT_Reversed; Digikey 650908-5 -> 609-86094648114H55V1LF-ND; LCSC (none) -> C464621
Connections:
- net ~{EXT_DTK}: now reaches J1.b28 (~{EXT_DTK})
- net ~{RESET}: now reaches J1.c12 (~{RESET})
- net ~{DTACK}: now reaches J1.c6 (~{DTACK})
- no-connect marks 17 -> 14
Changed lines of the file:
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@@
   (title_block
     (title "SEthernet PDS Ethernet Card for Macintosh SE")
-    (date "2023-11-10")
-    (rev "0")
+    (date "2024-01-27")
+    (rev "1")
   )
   (junction (at 73.66 30.48) (diameter 0) (color 0 0 0 0)
@@
   (no_connect (at 43.18 85.09))
   (no_connect (at 43.18 99.06))
-  (no_connect (at 99.06 114.3))
   (no_connect (at 43.18 87.63))
-  (no_connect (at 43.18 111.76))
   (no_connect (at 43.18 105.41))
   (no_connect (at 43.18 102.87))
   (no_connect (at 43.18 125.73))
   (no_connect (at 43.18 114.3))
-  (no_connect (at 99.06 116.84))
   (no_connect (at 43.18 116.84))
   (bus_entry (at 107.95 69.85) (size -2.54 2.54)
@@
     (stroke (width 0) (type default))
   )
+  (wire (pts (xy 43.18 111.76) (xy 33.02 111.76))
+    (stroke (width 0) (type default))
+  )
   (wire (pts (xy 35.56 77.47) (xy 43.18 77.47))
     (stroke (width 0) (type default))
@@
     (stroke (width 0) (type default))
   )
+  (wire (pts (xy 99.06 116.84) (xy 109.22 116.84))
+    (stroke (width 0) (type default))
+  )
   (bus (pts (xy 107.95 54.61) (xy 107.95 57.15))
     (stroke (width 0) (type default))
@@
   )
   (wire (pts (xy 99.06 74.93) (xy 105.41 74.93))
+    (stroke (width 0) (type default))
+  )
+  (wire (pts (xy 99.06 114.3) (xy 109.22 114.3))
     (stroke (width 0) (type default))
   )
@@
     )
   )
+  (global_label "~{EXT_DTK}" (shape output) (at 109.22 116.84 0) (fields_autoplaced)
+    (effects (font (size 1.27 1.27)) (justify left))
+    (property "Intersheetrefs" "${INTERSHEET_REFS}" (at 120.0065 116.84 0)
+      (effects (font (size 1.27 1.27)) (justify left) hide)
+    )
+  )
   (global_label "~{IPL1}" (shape input) (at 109.22 123.19 0) (fields_autoplaced)
     (effects (font (size 1.27 1.27)) (justify left))
@@
     )
   )
+  (global_label "~{DTACK}" (shape output) (at 109.22 114.3 0) (fields_autoplaced)
+    (effects (font (size 1.27 1.27)) (justify left))
+    (property "Intersheetrefs" "${INTERSHEET_REFS}" (at 118.0714 114.3 0)
+      (effects (font (size 1.27 1.27)) (justify left) hide)
+    )
+  )
   (global_label "~{LDS}" (shape output) (at 109.22 110.49 0) (fields_autoplaced)
     (effects (font (size 1.27 1.27)) (justify left))
@@
     (property "Intersheetrefs" "${INTERSHEET_REFS}" (at 116.2382 120.65 0)
       (effects (font (size 1.27 1.27)) (justify left) hide)
+    )
+  )
+  (global_label "~{RESET}" (shape input) (at 33.02 111.76 180) (fields_autoplaced)
+    (effects (font (size 1.27 1.27)) (justify right))
+    (property "Intersheetrefs" "${INTERSHEET_REFS}" (at 24.2897 111.76 0)
+      (effects (font (size 1.27 1.27)) (justify right) hide)
     )
   )
@@
   (symbol (lib_id "PDS-Ethernet:SE_PDS") (at 68.58 27.94 0) (unit 1)
     (in_bom yes) (on_board yes) (dnp no) (fields_autoplaced)
-    (property "Reference" "J1" (at 87.0459 135.89 0)
+    (property "Reference" "J1" (at 91.0941 29.21 0)
       (effects (font (size 1.27 1.27)) (justify left))
     )
-    (property "Value" "Macintosh SE PDS Interface" (at 87.0459 138.43 0)
+    (property "Value" "Macintosh SE PDS Interface" (at 91.0941 31.75 0)
       (effects (font (size 1.27 1.27)) (justify left))
     )
-    (property "Footprint" "Connector_DIN:DIN41612_C_3x32_Female_Vertical_THT" (at 177.8 21.59 0)
+    (property "Footprint" "PDS-Ethernet:DIN41612_C_3x32_Female_Vertical_THT_Reversed" (at 177.8 21.59 0)
       (effects (font (size 1.27 1.27)) hide)
     )
@@
       (effects (font (size 1.27 1.27)) hide)
     )
-    (property "Digikey" "650908-5" (at 68.58 27.94 0)
-      (effects (font (size 1.27 1.27)) hide)
-    )
+    (property "Digikey" "609-86094648114H55V1LF-ND" (at 68.58 27.94 0)
+      (effects (font (size 1.27 1.27)) hide)
+    )
+    (property "LCSC" "C464621" (at 68.58 27.94 0)
+      (effects (font (size 1.27 1.27)) hide)
+    )
