File: boards/se30/se30.kicad_pcb (KiCad board)
At the start: 2 copper layers, 116.8 x 59.7 mm, 43 parts, among them J1 Mac SE/30 PDS Interface, J2 Conn_02x05_Odd_Even, U1 ENC624J600-PT, U2 SST39SF010, U3 GAL16V8, U4 GAL16V8, U5 LD1117S33TR_SOT223, Y1 25MHz

Commit message: SE30 rev1
Parts:
- removed C10: 1uF, Capacitor_SMD:C_0805_2012Metric_Pad1.18x1.45mm_HandSolder
- removed the R4 at (49.1, 47.4)
- removed U5: LD1117S33TR_SOT223, Package_TO_SOT_SMD:SOT-223-3_TabPin2
- added J3: Conn_01x07, Connector_PinHeader_2.54mm:PinHeader_1x07_P2.54mm_Vertical, F.Cu at (139.7, 48.3)
- added J4: Mac SE/30 PDS Interface, PDS-Ethernet:DIN41612_C_3x40_Female_Horizontal_THT, F.Cu at (34.9, 30.5)
- added JP3: SolderJumper_2_Open, Jumper:SolderJumper-2_P1.3mm_Open_RoundedPad1.0x1.5mm, B.Cu at (128.9, 69.8)
- added R3: 10K, Resistor_SMD:R_0805_2012Metric_Pad1.20x1.40mm_HandSolder, F.Cu at (128.9, 69.8)
- added R6: 49.9, Resistor_SMD:R_0805_2012Metric_Pad1.20x1.40mm_HandSolder, F.Cu at (47.6, 54.6)
- U2: footprint Package_LCC:PLCC-32_THT-Socket -> Package_SO:TSOP-I-32_14.4x8mm_P0.5mm
- U3: value GAL16V8 -> ATF1502AS-xAx44; footprint Package_LCC:PLCC-20_THT-Socket -> Package_QFP:TQFP-44_10x10mm_P0.8mm
- U4: value GAL16V8 -> LD1117S33TR_SOT223; footprint Package_LCC:PLCC-20_THT-Socket -> Package_TO_SOT_SMD:SOT-223-3_TabPin2
- moved U4 95.1 mm to (36.0, 67.1)
- moved R4 61.5 mm to (121.3, 43.3), turned to -90 degrees
- moved R1 42.1 mm to (134.0, 69.8), turned to 90 degrees
- moved R2 41.9 mm to (131.5, 69.8), turned to 90 degrees
- moved C9 37.8 mm to (99.3, 43.3), turned to 90 degrees
- moved JP2 37.6 mm to (131.4, 69.8)
- moved JP1 37.4 mm to (134.0, 69.8)
- moved U3 26.3 mm to (118.1, 55.1), turned to -90 degrees
- moved U2 22.9 mm to (99.1, 55.4), turned to -90 degrees
- moved C8 17.3 mm to (115.7, 43.3), turned to 90 degrees
- moved C13 14.7 mm to (85.0, 52.7)
- moved C3 14.5 mm to (80.2, 51.4)
- moved C1 14.4 mm to (60.6, 49.3)
- moved C5 14.4 mm to (57.2, 52.1)
- moved C6 14.4 mm to (57.2, 54.8)
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- renumbered R3 to R1, R9 to R10, R10 to R11, R11 to R12, R4 to R2, R2 to R4, R1 to R5, R6 to R7, R7 to R8, R8 to R9
Connections:
- JP1 pad 2: Net-(JP1-B) -> /~{SLOTID_0}
- JP2 pad 2: Net-(JP2-B) -> /~{SLOTID_1}
- R1 pad 2: Net-(JP1-B) -> /~{SLOTID_0}
- R2 pad 2: Net-(JP2-B) -> /~{SLOTID_1}
- R4 pad 1: +3.3V -> GND
- U2 pad 1: GND -> A11
- U2 pad 10: A2 -> GND
- U2 pad 11: A1 -> A15
- U2 pad 12: A0 -> A12
- U2 pad 13: D24 -> A7
- U2 pad 14: D25 -> A6
- U2 pad 15: D26 -> A5
- U2 pad 16: GND -> A4
- U2 pad 17: D27 -> A3
- U2 pad 18: D28 -> A2
- U2 pad 19: D29 -> A1
- U2 pad 2: GND -> A9
- U2 pad 20: D30 -> A0
- U2 pad 21: D31 -> D24
- U2 pad 22: GND -> D25
- U2 pad 23: A10 -> D26
- U2 pad 24: /ROM_~{OE} -> GND
- U2 pad 25: A11 -> D27
- U2 pad 26: A9 -> D28
- U2 pad 27: A8 -> D29
- U2 pad 28: A13 -> D30
- U2 pad 29: A14 -> D31
- U2 pad 3: A15 -> A8
- U2 pad 31: /ROM_~{WE} -> A10
- U2 pad 32: +5V -> /ROM_~{OE}
- U2 pad 4: A12 -> A13
- U2 pad 5: A7 -> A14
- U2 pad 6: A6 -> GND
- U2 pad 7: A5 -> /ROM_~{WE}
- U2 pad 8: A4 -> +5V
- U2 pad 9: A3 -> GND
- U3 pad 1: Net-(JP2-B) -> /TDI
- U3 pad 10: GND -> /ROM_~{WE}
- U3 pad 11: A31 -> A0
- U3 pad 12: /ROM_~{CS} -> A16
- U3 pad 13: /ETH_CS -> A24
- U3 pad 14: /ETH_~{INT} -> A25
- U3 pad 15: ~{AS} -> A26
- U3 pad 16: A16 -> GND
- U3 pad 17: ~{IRQ3} -> +5V
- U3 pad 18: ~{IRQ2} -> A27
- U3 pad 19: ~{IRQ1} -> A28
- U3 pad 2: Net-(JP1-B) -> /ETH_~{INT}
- U3 pad 20: +5V -> A29
- U3 pad 3: A24 -> /ROM_~{OE}
- U3 pad 4: A25 -> GND
- U3 pad 5: A26 -> /B1SEL
- U3 pad 6: A27 -> /ETH_CS
- U3 pad 7: A28 -> /TMS
- U3 pad 8: A29 -> /B0SEL
- U3 pad 9: A30 -> +5V
- U4 pad 1: /ETH_CS -> GND
- U4 pad 2: /ROM_~{CS} -> +3.3V
- U4 pad 3: A0 -> +5V
Routing:
- net CPUCLK: track 0.00 -> 194.7 mm, vias 0 -> 1
- net +5V: track 249.5 -> 362.6 mm, vias 3 -> 6
- net GND: track 38.2 -> 143.4 mm, vias 64 -> 25
- net /PDS Interface/ECLK: track 0.00 -> 58.3 mm
- net /PDS Interface/C16M: track 0.00 -> 53.0 mm
- net D2: track 0.00 -> 52.3 mm
- net A23: track 0.00 -> 51.1 mm
- net D8: track 0.00 -> 51.0 mm
- net -12V: track 0.00 -> 50.9 mm
- net /PDS Interface/~{IPL2}: track 0.00 -> 50.9 mm
- net D5: track 0.00 -> 50.8 mm
- net D0: track 0.00 -> 50.7 mm
- net /PDS Interface/~{CIOUT}: track 0.00 -> 50.4 mm
- net A21: track 0.00 -> 50.3 mm
- net /PDS Interface/~{BUSLOCK}: track 0.00 -> 50.3 mm
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- added copper zone on In1.Cu, net GND
- added copper zone on In2.Cu, net GND
Other:
- copper layers 2 -> 4
- board text added: "+5V"
- board text added: "1 cycle (normal) 2 cycles (relaxed)"
- board text added: "10/100 Ethernet Card for 68030 PDS Slot github.com/rhalkyard/SEthernet"
- board text added: "9 (SE/30, IIsi) E (IIfx only) A (SE/30, IIsi) B (SE/30, IIsi)"
- board text added: "GND"
- board text added: "JP3"
- board text added: "Open Closed"
- board text added: "Revision 1"
- board text added: "Slot Address"
- board text added: "TCK"
- board text added: "TDI"
- board text added: "TDO"
- board text added: "TMS"
- board text added: "V_{PP}"
- board text added: "~{DSACK} Delay"
- board text removed: "10/100 Ethernet card for Macintosh SE/30 and IIsi github.com/rhalkyard/SEthernet"
- board text removed: "9 E A B"
- board text removed: "Address Decode"
- board text removed: "Bus Interface"
- board text removed: "Declaration ROM"
- board text removed: "Revision 0"
- board text removed: "Slot"
