File: boards/se30/se30.kicad_sch (KiCad schematic)
At the start: 42 parts, among them J3 Conn_02x05_Odd_Even, U1 ENC624J600-PT, U2 GAL16V8, U3 GAL16V8, U4 SST39SF010, U5 LD1117S33TR_SOT223, Y1 25MHz

Commit message: Schematic PDFs
Changed lines of the file:
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@@
     (stroke (width 0) (type default))
   )
-  (text_box "In 16-bit mode, A0..14 on the ENC624J600 addresses a *WORD*, rather than a byte."
-    (at 96.52 102.87 90) (size 7.62 36.83)
+  (text_box "Data bus is byte-swapped to preserve ordering of byte-wise addressing between little-endian ENC624J600 and big-endian 68K."
+    (at 96.52 55.88 90) (size 11.43 40.64)
     (stroke (width -0.0001) (type default))
     (fill (type none))
+    (effects (font (size 1.27 1.27)) (justify left top))
+  )
+  (text_box "In 16-bit mode, A0..14 on the ENC624J600 addresses a *WORD*, rather than a byte, so A1 on the PDS goes to A0 on the ENC624J600."
+    (at 95.25 101.6 90) (size 11.43 36.83)
+    (stroke (width -0.0001) (type default))
+    (fill (type none))

Commit message: SE30 rev1
Parts:
- removed C14: 1uF, Capacitor_SMD:C_0805_2012Metric_Pad1.18x1.45mm_HandSolder, symbol Device:C
- removed U2, U3: GAL16V8, Package_LCC:PLCC-20_THT-Socket, symbol Logic_Programmable:GAL16V8
- added J3: Conn_01x07, Connector_PinHeader_2.54mm:PinHeader_1x07_P2.54mm_Vertical, symbol Connector_Generic:Conn_01x07
- added JP3: SolderJumper_2_Open, Jumper:SolderJumper-2_P1.3mm_Open_RoundedPad1.0x1.5mm, symbol Jumper:SolderJumper_2_Open
- added R1: 10K, Resistor_SMD:R_0805_2012Metric_Pad1.20x1.40mm_HandSolder, symbol Device:R
- added U3: ATF1502AS-xAx44, Package_QFP:TQFP-44_10x10mm_P0.8mm, symbol CPLD_Microchip:ATF1502AS-xAx44
- U4: footprint Package_LCC:PLCC-32_THT-Socket -> Package_SO:TSOP-I-32_14.4x8mm_P0.5mm; symbol Memory_Flash:SST39SF010 -> PDS-Ethernet:SST39SF010-TSOP32
- renumbered R9 to R10, R10 to R11, R11 to R12, R2 to R4, R1 to R5, R4 to R6, R6 to R7, R7 to R8, R8 to R9, U5 to U4
Connections:
- net +3.3V: no longer R4.1
- net +5V: now also U4.8 (VCC), J3.5 (Pin_5), R1.1, U3.17 (VCC), U3.29 (VCC), U3.41 (VCC), U3.9 (VCC); no longer U4.32 (VCC)
- net A0: now also U4.20 (A0), U3.11 (I/O); no longer U4.12 (A0)
- net A1: now also U4.19 (A1); no longer U4.11 (A1)
- net A10: now also U4.31 (A10); no longer U4.23 (A10)
- net A11: now also U4.1 (A11); no longer U4.25 (A11)
- net A12: now also U4.12 (A12); no longer U4.4 (A12)
- net A13: now also U4.4 (A13); no longer U4.28 (A13)
- net A14: now also U4.5 (A14); no longer U4.29 (A14)
- net A15: now also U4.11 (A15); no longer U4.3 (A15)
- net A16: now also U3.12 (I/O)
- net A2: now also U4.18 (A2); no longer U4.10 (A2)
- net A24: now also U3.13 (I/O)
- net A25: now also U3.14 (I/O)
- net A26: now also U3.15 (I/O)
- net A27: now also U3.18 (I/O)
- net A28: now also U3.19 (I/O/PD2)
- net A29: now also U3.20 (I/O)
- net A3: now also U4.17 (A3); no longer U4.9 (A3)
- net A30: now also U3.21 (I/O)
- net A31: now also U3.22 (I/O)
- net A4: now also U4.16 (A4); no longer U4.8 (A4)
- net A5: now also U4.15 (A5); no longer U4.7 (A5)
- net A6: now also U4.14 (A6); no longer U4.6 (A6)
- net A7: now also U4.13 (A7); no longer U4.5 (A7)
- net A8: now also U4.3 (A8); no longer U4.27 (A8)
- net A9: now also U4.2 (A9); no longer U4.26 (A9)
- net B0SEL: now also U3.8 (I/O)
- net B1SEL: now also U3.5 (I/O/PD1)
- net D24: now also U4.21 (D0); no longer U4.13 (D0)
- net D25: now also U4.22 (D1); no longer U4.14 (D1)
- net D26: now also U4.23 (D2); no longer U4.15 (D2)
- net D27: now also U4.25 (D3); no longer U4.17 (D3)
- net D28: now also U4.26 (D4); no longer U4.18 (D4)
- net D29: now also U4.27 (D5); no longer U4.19 (D5)
- net D30: now also U4.28 (D6); no longer U4.20 (D6)
- net D31: now also U4.29 (D7); no longer U4.21 (D7)
- net ETH_CS: now also U3.6 (I/O)
- net ETH_~{INT}: now also U3.2 (I/O)
- net GND: now also R4.1, U4.10 (A16), U4.24 (GND), U4.6 (NC), U4.9 (NC), J3.6 (Pin_6), JP3.1 (A), U3.16 (GND), U3.24 (GND), U3.36 (GND), U3.4 (GND); no longer U4.1 (NC), U4.16 (GND), U4.2 (A16), U4.22 (CE)
- net ROM_~{OE}: now also U4.32 (OE), U3.3 (I/O); no longer U4.24 (OE)
- net ROM_~{WE}: now also U4.7 (PGM), U3.10 (I/O); no longer U4.31 (PGM)
- net R/~{W}: now also U3.28 (I/O)
- net SIZ0: now also U3.25 (I/O)
- net SIZ1: now also U3.27 (I/O)
- net ~{AS}: now also U3.23 (I/O)
- net ~{DSACK0}: now also U3.30 (I/O)
- net ~{DSACK1}: now also U3.31 (I/O)
- net ~{DS}: now also U3.33 (I/O)
- net ~{IRQ1}: now also U3.44 (I/O)
- net ~{IRQ2}: now also U3.43 (I/O)
- net ~{IRQ3}: now also U3.42 (I/O)
- net ~{SLOTID_1}: now reaches JP2.2 (B), R1.2
- net ~{SLOTID_1}: now also U3.34 (I/O)
- net ~{SLOTID_0}: now reaches JP1.2 (B), R2.2
- net ~{SLOTID_0}: now also U3.35 (I/O/GCLK3)
- new net CPLD_VPP: J3.7 (Pin_7), U3.38 (I/OE1/Vpp)
- new net CPUCLK: U3.40 (I/OE2/GCLK2)
- new net TCK: J3.2 (Pin_2), U3.26 (I/O/TCK)
- new net TDI: J3.3 (Pin_3), U3.1 (I/O/TDI)
- new net TDO: J3.4 (Pin_4), U3.32 (I/O/TDO)
- new net TMS: J3.1 (Pin_1), U3.7 (I/O/TMS)
- new net WAITCTL: JP3.2 (B), R1.2, U3.37 (I/GCLK1)
- no-connect marks 3 -> 2
Other:
- note removed: "X = open O = closed XX: Slot 9, IRQ 1 XO: Slot E, IRQ 1 OX: Slot A, IRQ 2 XX: Slot B, IRQ 3"
- moved on the sheet: JP1, JP2, R1, R2, R4
