File: boards/breakout/breakout.kicad_sch (KiCad schematic)
At the start: 12 parts, among them J1 8P8C_Shielded, J2 DE15_Receptacle_HighDensity_M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, J3 Conn_02x04_Odd_Even, J4 Conn_02x05_Odd_Even

Commit message: Rev1 hardware
Parts:
- JP1, JP2: symbol Jumper:Jumper_2_Bridged -> Jumper:Jumper_2_Open
- R1, R2: footprint Resistor_SMD:R_0805_2012Metric_Pad1.20x1.40mm_HandSolder -> Resistor_THT:R_Axial_DIN0204_L3.6mm_D1.6mm_P7.62mm_Horizontal; Digikey RMCF0805FT180R -> CF18JT180R
Changed lines of the file:
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@@
   (title_block
     (title "Breakout board for SEthernet-series PDS Ethernet cards")
-    (date "2023-11-10")
-    (rev "0")
+    (date "2024-01-27")
+    (rev "1")
   )
   (junction (at 87.63 71.12) (diameter 0) (color 0 0 0 0)
@@
     (effects (font (size 1.27 1.27)) (justify right bottom))
   )
-  (symbol (lib_id "Jumper:Jumper_2_Bridged") (at 193.04 76.2 0) (unit 1)
+  (symbol (lib_id "Jumper:Jumper_2_Open") (at 193.04 76.2 0) (unit 1)
     (in_bom yes) (on_board yes) (dnp no) (fields_autoplaced)
     (property "Reference" "JP2" (at 193.04 71.12 0)
@@
     )
     (property "Value" "Jumper_2_Bridged" (at 193.04 73.66 0)
-      (effects (font (size 1.27 1.27)))
+      (effects (font (size 1.27 1.27)) hide)
     )
     (property "Footprint" "Connector_PinHeader_2.54mm:PinHeader_1x02_P2.54mm_Vertical" (at 193.04 76.2 0)
@@
     )
   )
-  (symbol (lib_id "Jumper:Jumper_2_Bridged") (at 193.04 68.58 0) (unit 1)
+  (symbol (lib_id "Jumper:Jumper_2_Open") (at 193.04 68.58 0) (unit 1)
     (in_bom yes) (on_board yes) (dnp no) (fields_autoplaced)
     (property "Reference" "JP1" (at 193.04 63.5 0)
@@
     )
     (property "Value" "Jumper_2_Bridged" (at 193.04 66.04 0)
-      (effects (font (size 1.27 1.27)))
+      (effects (font (size 1.27 1.27)) hide)
     )
     (property "Footprint" "Connector_PinHeader_2.54mm:PinHeader_1x02_P2.54mm_Vertical" (at 193.04 68.58 0)
@@
       (effects (font (size 1.27 1.27)))
     )
-    (property "Footprint" "Resistor_SMD:R_0805_2012Metric_Pad1.20x1.40mm_HandSolder" (at 76.2 69.342 90)
+    (property "Footprint" "Resistor_THT:R_Axial_DIN0204_L3.6mm_D1.6mm_P7.62mm_Horizontal" (at 76.2 69.342 90)
       (effects (font (size 1.27 1.27)) hide)
     )
@@
       (effects (font (size 1.27 1.27)) hide)
     )
-    (property "Digikey" "RMCF0805FT180R" (at 76.2 71.12 0)
+    (property "Digikey" "CF18JT180R" (at 76.2 71.12 0)
       (effects (font (size 1.27 1.27)) hide)
     )
@@
       (effects (font (size 1.27 1.27)))
     )
-    (property "Footprint" "Resistor_SMD:R_0805_2012Metric_Pad1.20x1.40mm_HandSolder" (at 76.2 64.262 90)
+    (property "Footprint" "Resistor_THT:R_Axial_DIN0204_L3.6mm_D1.6mm_P7.62mm_Horizontal" (at 76.2 64.262 90)
       (effects (font (size 1.27 1.27)) hide)
     )
@@
       (effects (font (size 1.27 1.27)) hide)
     )
-    (property "Digikey" "RMCF0805FT180R" (at 76.2 66.04 0)
-      (effects (font (size 1.27 1.27)) hide)
-    )
+    (property "Digikey" "CF18JT180R" (at 76.2 66.04 0)
+      (effects (font (size 1.27 1.27)) hide)
+    )

Commit message: Breakout: use threaded inserts for mounting
Resize mounting holes for use with Wurth 9774025360R threaded inserts.
Parts:
- H1, H2: footprint PDS-Ethernet:MountingHole_3.5mm_Pad -> PDS-Ethernet:Wurth_9774025360R; Digikey (none) -> 9774025360R
Changed lines of the file:
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@@
       (effects (font (size 1.27 1.27)) (justify left))
     )
-    (property "Footprint" "PDS-Ethernet:MountingHole_3.5mm_Pad" (at 35.56 97.79 0)
+    (property "Footprint" "PDS-Ethernet:Wurth_9774025360R" (at 35.56 97.79 0)
       (effects (font (size 1.27 1.27)) hide)
     )
     (property "Datasheet" "~" (at 35.56 97.79 0)
+      (effects (font (size 1.27 1.27)) hide)
+    )
+    (property "Digikey" "9774025360R" (at 35.56 97.79 0)
       (effects (font (size 1.27 1.27)) hide)
     )
@@
       (effects (font (size 1.27 1.27)) (justify left))
     )
-    (property "Footprint" "PDS-Ethernet:MountingHole_3.5mm_Pad" (at 62.23 97.79 0)
+    (property "Footprint" "PDS-Ethernet:Wurth_9774025360R" (at 62.23 97.79 0)
       (effects (font (size 1.27 1.27)) hide)
     )
@@
       (effects (font (size 1.27 1.27)) hide)
     )
+    (property "Digikey" "9774025360R" (at 62.23 97.79 0)
+      (effects (font (size 1.27 1.27)) hide)
+    )
